File: pcb/hackboard.kicad_pcb (KiCad board)
At the start: 2 copper layers, 309.7 x 117.3 mm, 255 parts, among them SW1 SW_Push_45deg, SW10 SW_Push_45deg, SW11 SW_Push_45deg, SW12 SW_Push_45deg, SW13 SW_Push_45deg, SW14 SW_Push_45deg, SW15 SW_Push_45deg, SW16 SW_Push_45deg, SW17 SW_Push_45deg, SW18 SW_Push_45deg, SW19 SW_Push_45deg, SW2 SW_Push_45deg, SW20 SW_Push_45deg, SW21 SW_Push_45deg, SW22 SW_Push_45deg, SW23 SW_Push_45deg, SW24 SW_Push_45deg, SW25 SW_Push_45deg, SW26 SW_Push_45deg, SW27 SW_Push_45deg, SW28 SW_Push_45deg, SW29 SW_Push_45deg, SW3 SW_Push_45deg, SW30 SW_Push_45deg, SW31 SW_Push_45deg, SW32 SW_Push_45deg, SW33 SW_Push_45deg, SW34 SW_Push_45deg, SW35 SW_Push_45deg, SW36 SW_Push_45deg, SW37 SW_Push_45deg, SW38 SW_Push_45deg, SW39 SW_Push_45deg, SW4 SW_Push_45deg, SW40 SW_Push_45deg, SW41 SW_Push_45deg, SW42 SW_Push_45deg, SW43 SW_Push_45deg, SW44 SW_Push_45deg, SW45 SW_Push_45deg, SW46 SW_Push_45deg, SW47 SW_Push_45deg, SW48 SW_Push_45deg, SW49 SW_Push_45deg, SW5 SW_Push_45deg, SW50 SW_Push_45deg, SW51 SW_Push_45deg, SW52 SW_Push_45deg, SW53 SW_Push_45deg, SW54 SW_Push_45deg, SW55 SW_Push_45deg, SW56 SW_Push_45deg, SW57 SW_Push_45deg, SW58 SW_Push_45deg, SW59 SW_Push_45deg, SW6 SW_Push_45deg, SW60 SW_Push_45deg, SW61 SW_Push_45deg, SW62 SW_Push_45deg, SW63 SW_Push_45deg, SW64 SW_Push_45deg, SW65 SW_Push_45deg, SW66 SW_Push_45deg, SW67 SW_Push_45deg, SW68 SW_Push_45deg, SW69 SW_Push_45deg, SW7 SW_Push_45deg, SW70 SW_Push_45deg, SW71 SW_Push_45deg, SW72 SW_Push_45deg, SW73 SW_Push_45deg, SW74 SW_Push_45deg, SW75 SW_Push_45deg, SW76 SW_Push_45deg, SW77 SW_Push_45deg, SW78 SW_Push_45deg, SW79 SW_Push_45deg, SW8 SW_Push_45deg, SW80 SW_Push_45deg, SW81 SW_Push_45deg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

Commit message: modified:   pcb/hackboard.kicad_pcb 	modified:   pcb/hackboard.kicad_prl 	modified:   pcb/hackboard.kicad_sch 	modified:   pcb/production/bom.csv 	modified:   pcb/production/hackboard.zip 	modified:   pcb/production/netlist.ipc 	modified:   pcb/production/positions.csv
Parts:
- D1, D10, D11, D12, D13, D14, D15, D16, D17, D18, D19, D2, D20, D21, D22, D23, D24, D25, D26, D27, D28, D29, D3, D30, D31, D32, D33, D34, D35, D36, D37, D38, D39, D4, D40, D41, D42, D43, D44, D45, D46, D47, D48, D49, D5, D50, D51, D52, D53, D54, D55, D56, D57, D58, D59, D6, D60, D61, D62, D63, D64, D65, D66, D67, D68, D69, D7, D70, D71, D72, D73, D74, D75, D76, D77, D78, D79, D8, D80, D81, D82, D9: footprint customDiode:D_0402_1005Metric_Pad0.77x0.64mm_HandSolder-withVia -> Diode_SMD:D_SOD-123
- moved D109 322.1 mm to (230.4, 78.3)
- moved D11 322.1 mm to (206.6, 62.3)
- moved D137 322.1 mm to (206.6, 116.4)
- moved D152 322.1 mm to (242.3, 135.4)
- moved D161 322.1 mm to (230.4, 154.5)
- moved D164 322.1 mm to (289.9, 156.9)
- moved D27 322.1 mm to (230.4, 81.3)
- moved D55 322.1 mm to (206.6, 119.4)
- moved D70 322.1 mm to (242.3, 138.5)
- moved D79 322.1 mm to (230.4, 157.5)
- moved D82 322.1 mm to (289.9, 159.9)
- moved D93 322.1 mm to (206.6, 59.2)
- moved SW10 322.1 mm to (190.0, 49.1)
- moved SW13 322.1 mm to (247.2, 49.1)
- moved SW26 322.1 mm to (213.9, 68.1)
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Connections:
- U2 pad 19: COL10 -> COL15
- U2 pad 20: COL9 -> COL14
- U2 pad 22: COL14 -> ROW1
- U2 pad 23: COL15 -> ROW2
- U2 pad 24: unconnected-(U2-GPA7-Pad24) -> ROW3
- U4 pad 1: COL2 -> COL3
- U4 pad 2: COL1 -> COL2
- U4 pad 20: ROW3 -> unconnected-(U4-GPA3-Pad20)
- U4 pad 21: ROW2 -> unconnected-(U4-GPA4-Pad21)
- U4 pad 22: ROW1 -> COL10
- U4 pad 23: COL8 -> COL9
- U4 pad 24: COL7 -> COL8
- U4 pad 25: COL6 -> COL7
- U4 pad 26: COL5 -> COL6
- U4 pad 27: COL4 -> COL5
- U4 pad 28: COL3 -> COL4
- U4 pad 3: unconnected-(U4-GPB6-Pad3) -> COL1
Routing:
- net GND: track 23.7 -> 151.4 mm, vias 105 -> 104
- net ROW1: track 282.5 -> 351.0 mm, vias 1 -> 15
- net VCC: track 345.3 -> 291.2 mm, vias 7 -> 8
- net COL10: track 169.0 -> 200.9 mm, vias 0 -> 1
- net ROW2: track 325.0 -> 355.2 mm, vias 2 -> 17
- net ROW4: track 313.3 -> 335.2 mm, vias 1 -> 15
- net ROW5: track 332.2 -> 351.8 mm, vias 2 -> 16
- net SCL: track 305.9 -> 287.4 mm
- net SDA: track 306.0 -> 288.9 mm, vias 2 -> 3
- net +5V: track 31.2 -> 48.1 mm, vias 5 -> 18
- net SPACE_DIN: track 126.0 -> 113.3 mm
- net COL8: track 131.9 -> 141.1 mm, vias 0 -> 1
- net COL12: track 123.6 -> 132.4 mm
- net COL7: track 113.7 -> 122.0 mm, vias 0 -> 1
- net COL11: track 150.8 -> 159.0 mm
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